Commit message: modified:   config/address.yaml 	modified:   config/camera.yaml 	deleted:    models/__init__.py 	deleted:    models/finger_net.py 	modified:   modules/__init__.py 	new file:   modules/finger/def_node.txt 	new file:   modules/finger/surf_coor.txt 	new file:   modules/finger/surf_node.txt 	new file:   modules/finger/surf_tri.txt 	deleted:    modules/protobuf/cam_msg.proto 	new file:   modules/protobuf/finger_msg.proto 	renamed:    modules/protobuf/cam_msg_pb2.py -> modules/protobuf/finger_msg_pb2.py 	modified:   modules/protobuf/generate_pb.sh 	modified:   modules/protobuf/robot_msg.proto 	modified:   modules/protobuf/robot_msg_pb2.py 	modified:   modules/robotiq/arg85/arg85.urdf 	modified:   requirements.txt 	modified:   rerun_loader_urdf.py 	modified:   server.py 	new file:   test.py

File: modules/robotiq/arg85/arg85.urdf (robot description, URDF)
Before this commit: robot robotiq_arg85, 9 links, 8 joints
Links:
- link left_inner_finger: geometry collision mesh filename=meshes/inner_finger_coarse.STL; visual mesh filename=meshes/inner_finger_fine.STL
- link left_inner_knuckle: geometry collision mesh filename=meshes/inner_knuckle_coarse.STL; visual mesh filename=meshes/inner_knuckle_fine.STL
- link left_outer_finger: geometry collision mesh filename=meshes/outer_finger_coarse.STL; visual mesh filename=meshes/outer_finger_fine.STL
- link left_outer_knuckle: geometry collision mesh filename=meshes/outer_knuckle_coarse.STL; visual mesh filename=meshes/outer_knuckle_fine.STL
- link right_inner_finger: geometry collision mesh filename=meshes/inner_finger_coarse.STL; visual mesh filename=meshes/inner_finger_fine.STL
- link right_inner_knuckle: geometry collision mesh filename=meshes/inner_knuckle_coarse.STL; visual mesh filename=meshes/inner_knuckle_fine.STL
- link right_outer_finger: geometry collision mesh filename=meshes/outer_finger_coarse.STL; visual mesh filename=meshes/outer_finger_fine.STL
- link right_outer_knuckle: geometry collision mesh filename=meshes/outer_knuckle_coarse.STL; visual mesh filename=meshes/outer_knuckle_fine.STL
- link robotiq_85_base_link: geometry collision mesh filename=meshes/robotiq_85_base_link_coarse.STL; visual mesh filename=meshes/robotiq_85_base_link_fine.STL
